File: breakout/breakout.kicad_pcb (KiCad board)
At the start: 2 copper layers, 68 x 48 mm, 9 parts, among them J1 Glasgow, J2 ScrewTerminals, J3 SignalsMale, J4 SignalsFemale, J5 SignalsMale, J6 SignalsFemale, J7 TestPoints

Commit message: [wip] add connector for generic fx2 logic analyzers
Parts:
- added J9: FX2LA, Connector_PinSocket_2.54mm:PinSocket_2x05_P2.54mm_Vertical, F.Cu at (129.5, 81.5)
- moved H1 11.0 mm to (189.0, 66.0)
- moved H2 11.0 mm to (189.0, 106.0)
- moved J1 11.0 mm to (133.5, 75.0)
- moved J2 11.0 mm to (181.0, 72.3)
- moved J3 11.0 mm to (148.5, 74.9)
- moved J4 11.0 mm to (143.5, 74.9)
- moved J5 11.0 mm to (153.5, 75.0)
- moved J6 11.0 mm to (158.5, 74.9)
- moved J7 11.0 mm to (168.5, 77.5)
Routing:
- net /D7: track 48.6 -> 59.2 mm
- net /D1: track 48.6 -> 57.4 mm
- net /D5: track 48.6 -> 57.1 mm
- net /D3: track 48.6 -> 55.7 mm
- net /D0: track 48.6 -> 54.9 mm
- net /D6: track 48.6 -> 54.1 mm
- net /D2: track 48.6 -> 53.2 mm
- net /D4: track 48.6 -> 53.0 mm
- net GND: vias 156 -> 155
Other:
- board size 68 x 48 mm -> 75 x 48 mm
